Commit message: [CHANGED] Poses of models to Unity coordenates

File: WorldParser/models/urdf/RoCKIn@Home.urdf (robot description, URDF)
Before this commit: robot RoCKIn@Home, 13 links, 0 joints
Links:
- added link RoCKInATHome__Wall_15, mass 0; collision box size=1.41579 0.2 2.5; visual box size=1.41579 0.2 2.5
- added link RoCKInATHome__Wall_17, mass 0; collision box size=1 0.2 0.5; visual box size=1 0.2 0.5
- link RoCKInATHome__Wall_14: geometry collision box size=1.18422 0.2 2.5; visual box size=1.18422 0.2 2.5

Commit message: [CHANGED] Coordenates of all origin tags

File: WorldParser/models/urdf/RoCKIn@Home.urdf (robot description, URDF)
Before this commit: robot RoCKIn@Home, 15 links, 0 joints
Joints:
- added joint joint_1: type fixed, parent RoCKInATHome__Wall_12, child RoCKInATHome__Wall_14
- added joint joint_10: type fixed, parent RoCKInATHome__Wall_12, child RoCKInATHome__Wall_30
- added joint joint_11: type fixed, parent RoCKInATHome__Wall_12, child RoCKInATHome__Wall_32
- added joint joint_12: type fixed, parent RoCKInATHome__Wall_12, child RoCKInATHome__Wall_35
- added joint joint_13: type fixed, parent RoCKInATHome__Wall_12, child RoCKInATHome__Wall_8
- added joint joint_2: type fixed, parent RoCKInATHome__Wall_12, child RoCKInATHome__Wall_15
- added joint joint_3: type fixed, parent RoCKInATHome__Wall_12, child RoCKInATHome__Wall_17
- added joint joint_4: type fixed, parent RoCKInATHome__Wall_12, child RoCKInATHome__Wall_18
- added joint joint_5: type fixed, parent RoCKInATHome__Wall_12, child RoCKInATHome__Wall_2
- added joint joint_6: type fixed, parent RoCKInATHome__Wall_12, child RoCKInATHome__Wall_20
- added joint joint_7: type fixed, parent RoCKInATHome__Wall_12, child RoCKInATHome__Wall_22
- added joint joint_8: type fixed, parent RoCKInATHome__Wall_12, child RoCKInATHome__Wall_24
- added joint joint_9: type fixed, parent RoCKInATHome__Wall_12, child RoCKInATHome__Wall_28
